File: GNSS.kicad_sch (KiCad schematic)
At the start: 19 parts, among them J10 USB_C_USB2.0_16P, J11 Micro_SD_Card, SW3 SW_GNSS, U6 NEO-M9N

Commit message: init v1.0.2
Parts:
- removed TP1: nSAFEBOOT, TestPoint:TestPoint_Pad_D1.0mm, symbol Connector:TestPoint
- added TP61, TP62, TP63, TP64, TP65: TestPoint, symbol Connector:TestPoint
- renumbered C60 to C61, C61 to C62, C62 to C63, C67 to C64, J10 to J61, J11 to J62, JP1 to JP61, L67 to L61, R62 to R61, R63 to R62, R67 to R63, R60 to R64, R61 to R65, R64 to R66, SW3 to SW61, U6 to U61
Connections:
- net SPI_CS0: now also J62.2 (DAT3/CD); no longer U61.18 (SDA/~{SPI_CS})
- net SPI_CS1: now also U61.18 (SDA/~{SPI_CS}); no longer J62.2 (DAT3/CD)
- net DAT2: now reaches J62.1 (DAT2)
- net DAT2: now also TP65.1
- net DAT1: now reaches J62.8 (DAT1)
- net DAT1: now also TP64.1
- net LNA_EN: now reaches U61.14 (LNA_EN)
- net LNA_EN: now also TP63.1
- net TIMEPULSE: now reaches U61.3 (TIMEPULSE)
- net TIMEPULSE: now also TP61.1
- net EXTINT: now reaches U61.4 (EXTINT)
- net EXTINT: now also TP62.1
- no-connect marks 8 -> 3

Commit message: v1.0.2 changelog
Parts:
- added TP63: TestPoint, TestPoint:TestPoint_THTPad_D1.5mm_Drill0.7mm, symbol Connector:TestPoint
- SW61: footprint Button_Switch_SMD:SW_SPST_B3U-1000P -> Button_Switch_SMD:SW_Push_1P1T_NO_CK_KMR2
- TP61, TP62: footprint (none) -> TestPoint:TestPoint_THTPad_D1.5mm_Drill0.7mm
- TP64: renamed from TP63; footprint (none) -> TestPoint:TestPoint_THTPad_D1.5mm_Drill0.7mm
- TP65: renamed from TP64; footprint (none) -> TestPoint:TestPoint_THTPad_D1.5mm_Drill0.7mm
- TP66: renamed from TP65; footprint (none) -> TestPoint:TestPoint_THTPad_D1.5mm_Drill0.7mm
Connections:
- net ~{SAFEBOOT}: now reaches U61.1 (~{SAFEBOOT})
- net ~{SAFEBOOT}: now also TP63.1
Other:
- moved on the sheet: TP61, TP62
Changed lines of the file:
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@@
 	(wire
 		(pts
-			(xy 165.1 38.1) (xy 167.64 38.1)
+			(xy 165.1 31.75) (xy 167.64 31.75)
 		)
 		(stroke
@@
 	(wire
 		(pts
-			(xy 100.33 96.52) (xy 91.44 96.52)
-		)
-		(stroke
-			(width 0)
-			(type default)
-		)
-	)
-	(wire
-		(pts
 			(xy 91.44 63.5) (xy 90.17 63.5)
 		)
@@
 	(wire
 		(pts
-			(xy 165.1 44.45) (xy 167.64 44.45)
+			(xy 165.1 38.1) (xy 167.64 38.1)
 		)
 		(stroke
@@
 	(wire
 		(pts
+			(xy 165.1 44.45) (xy 167.64 44.45)
+		)
+		(stroke
+			(width 0)
+			(type default)
+		)
+	)
+	(wire
+		(pts
 			(xy 113.03 58.42) (xy 115.57 58.42)
 		)
@@
 		)
 	)
+	(label "~{SAFEBOOT}"
+		(at 100.33 96.52 180)
+		(effects
+			(font
+				(size 1.27 1.27)
+			)
+			(justify right bottom)
+		)
+	)
 	(label "USB2_D-"
 		(at 49.53 53.34 0)
@@
 		)
 	)
+	(label "~{SAFEBOOT}"
+		(at 167.64 44.45 0)
+		(effects
+			(font
+				(size 1.27 1.27)
+			)
+			(justify left bottom)
+		)
+	)
 	(label "LNA_EN"
 		(at 135.89 78.74 0)
@@
 	)
 	(label "EXTINT"
-		(at 167.64 44.45 0)
+		(at 167.64 38.1 0)
 		(effects
 			(font
@@
 	)
 	(label "TIMEPULSE"
-		(at 167.64 38.1 0)
+		(at 167.64 31.75 0)
 		(effects
 			(font
@@
 	)
 	(symbol
+		(lib_id "Connector:TestPoint")
+		(at 165.1 44.45 0)
+		(mirror y)
+		(unit 1)
+		(exclude_from_sim no)
+		(in_bom yes)
+		(on_board yes)
+		(dnp no)
+		(property "Reference" "TP63"
+			(at 162.56 39.8779 0)
+			(effects
+				(font
+					(size 1.27 1.27)
+				)
+				(justify left)
+			)
+		)
+		(property "Value" "TestPoint"
+			(at 162.56 42.4179 0)
+			(effects
+				(font
+					(size 1.27 1.27)
+				)
+				(justify left)
+			)
+		)
+		(property "Footprint" "TestPoint:TestPoint_THTPad_D1.5mm_Drill0.7mm"
+			(at 160.02 44.45 0)
+			(effects
+				(font
+					(size 1.27 1.27)
+				)
+				(hide yes)
+			)
+		)
+		(property "Datasheet" "~"
+			(at 160.02 44.45 0)
+			(effects
+				(font
+					(size 1.27 1.27)
+				)
+				(hide yes)
+			)
+		)
+		(property "Description" "test point"
+			(at 165.1 44.45 0)
+			(effects
+				(font
+					(size 1.27 1.27)
+				)
+				(hide yes)
+			)
+		)
+		(pin "1"
+		)
+		(instances
+			(project "BLV_PCB"
+				(path "/e98ed281-6a46-49b2-ab41-e3d95fdf6973/e5b94b9f-016b-443f-970f-ae0598cc0fac"
+					(reference "TP63")
+					(unit 1)
+				)
+			)
+		)
+	)
+	(symbol
 		(lib_name "GND_3")
 		(lib_id "power:GND")
@@
 			)
 		)
-		(property "Footprint" "Button_Switch_SMD:SW_SPST_B3U-1000P"
+		(property "Footprint" "Button_Switch_SMD:SW_Push_1P1T_NO_CK_KMR2"
 			(at 76.2 93.98 0)
 			(effects
@@
 		(on_board yes)
 		(dnp no)
-		(property "Reference" "TP65"
+		(property "Reference" "TP66"
 			(at 73.66 147.8279 0)
 			(effects
@@
 			)
 		)
-		(property "Footprint" ""
+		(property "Footprint" "TestPoint:TestPoint_THTPad_D1.5mm_Drill0.7mm"
 			(at 71.12 152.4 0)
 			(effects
@@
 			(project "BLV_PCB"
 				(path "/e98ed281-6a46-49b2-ab41-e3d95fdf6973/e5b94b9f-016b-443f-970f-ae0598cc0fac"
-					(reference "TP65")
+					(reference "TP66")
 					(unit 1)
 				)
@@
 	(symbol
 		(lib_id "Connector:TestPoint")
-		(at 165.1 44.45 0)
+		(at 165.1 38.1 0)
 		(mirror y)
 		(unit 1)
@@
 		(dnp no)
 		(property "Reference" "TP62"
-			(at 162.56 39.8779 0)
+			(at 162.56 33.5279 0)
 			(effects
 				(font
@@
 		)
 		(property "Value" "TestPoint"
-			(at 162.56 42.4179 0)
+			(at 162.56 36.0679 0)
 			(effects
 				(font
@@
 			)
 		)
-		(property "Footprint" ""
-			(at 160.02 44.45 0)
+		(property "Footprint" "TestPoint:TestPoint_THTPad_D1.5mm_Drill0.7mm"
+			(at 160.02 38.1 0)
 			(effects
 				(font
@@
 		)
 		(property "Datasheet" "~"
-			(at 160.02 44.45 0)
+			(at 160.02 38.1 0)
 			(effects
 				(font
@@
 		)
 		(property "Description" "test point"
-			(at 165.1 44.45 0)
+			(at 165.1 38.1 0)
 			(effects
 				(font
@@
 	(symbol
 		(lib_id "Connector:TestPoint")
-		(at 165.1 38.1 0)
+		(at 165.1 31.75 0)
 		(mirror y)
 		(unit 1)
@@
 		(dnp no)
 		(property "Reference" "TP61"
-			(at 162.56 33.5279 0)
+			(at 162.56 27.1779 0)
 			(effects
 				(font
@@
 		)
 		(property "Value" "TestPoint"
-			(at 162.56 36.0679 0)
+			(at 162.56 29.7179 0)
 			(effects
 				(font
@@
 			)
 		)
-		(property "Footprint" ""
-			(at 160.02 38.1 0)
+		(property "Footprint" "TestPoint:TestPoint_THTPad_D1.5mm_Drill0.7mm"
+			(at 160.02 31.75 0)
 			(effects
 				(font
@@
 		)
 		(property "Datasheet" "~"
-			(at 160.02 38.1 0)
+			(at 160.02 31.75 0)
 			(effects
 				(font
@@
 		)
 		(property "Description" "test point"
-			(at 165.1 38.1 0)
+			(at 165.1 31.75 0)
 			(effects
 				(font
@@
 			)
 		)
-		(property "Datasheet" "https://www.we-online.com/components/products/datasheet/693072010801.pdf"
+		(property "Datasheet" ""
 			(at 119.38 166.37 0)
 			(effects
@@
 			)
 		)
-		(property "Description" "Micro SD Card Socket | https://elm-chan.org/docs/mmc/mmc_e.html"
+		(property "Description" ""
 			(at 119.38 166.37 0)
 			(effects
@@
 		)
 		(instances
-			(project "BLV_PCB"
+			(project ""
+				(path "/e98ed281-6a46-49b2-ab41-e3d95fdf6973/6e201a35-d390-4e65-a234-b842b3106670"
+					(reference "J62")
+					(unit 1)
+				)
 				(path "/e98ed281-6a46-49b2-ab41-e3d95fdf6973/e5b94b9f-016b-443f-970f-ae0598cc0fac"
 					(reference "J62")
@@
 		(on_board yes)
 		(dnp no)
-		(property "Reference" "TP64"
+		(property "Reference" "TP65"
 			(at 73.66 141.4779 0)
 			(effects
@@
 			)
 		)
-		(property "Footprint" ""
+		(property "Footprint" "TestPoint:TestPoint_THTPad_D1.5mm_Drill0.7mm"
 			(at 71.12 146.05 0)
 			(effects
@@
 			(project "BLV_PCB"
 				(path "/e98ed281-6a46-49b2-ab41-e3d95fdf6973/e5b94b9f-016b-443f-970f-ae0598cc0fac"
-					(reference "TP64")
+					(reference "TP65")
 					(unit 1)
 				)
@@
 		(on_board yes)
 		(dnp no)
-		(property "Reference" "TP63"
+		(property "Reference" "TP64"
 			(at 162.56 46.2279 0)
 			(effects
@@
 			)
 		)
-		(property "Footprint" ""
+		(property "Footprint" "TestPoint:TestPoint_THTPad_D1.5mm_Drill0.7mm"
 			(at 160.02 50.8 0)
 			(effects
@@
 			(project "BLV_PCB"
 				(path "/e98ed281-6a46-49b2-ab41-e3d95fdf6973/e5b94b9f-016b-443f-970f-ae0598cc0fac"
-					(reference "TP63")
+					(reference "TP64")
 					(unit 1)
 				)

Commit message: safepoint
Parts:
- C61: value 10uF -> 10u
- C62: value 1uF -> 1u
- L61: footprint Inductor_SMD:L_0201_0603Metric -> Inductor_SMD:L_0402_1005Metric
- SW61: value SW_GNSS -> KMR2
Changed lines of the file:
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@@
 			)
 		)
-		(property "Value" "SW_GNSS"
+		(property "Value" "KMR2"
 			(at 76.2 100.838 0)
 			(effects
@@
 			)
 		)
-		(property "Value" "1uF"
+		(property "Value" "1u"
 			(at 87.122 30.48 0)
 			(effects
@@
 			)
 		)
-		(property "Footprint" "Inductor_SMD:L_0201_0603Metric"
+		(property "Footprint" "Inductor_SMD:L_0402_1005Metric"
 			(at 152.4 73.66 0)
 			(effects
@@
 			)
 		)
-		(property "Value" "10uF"
+		(property "Value" "10u"
 			(at 75.692 30.48 0)
 			(effects
