File: BLV_PCB.kicad_pcb (KiCad board)
At the start: 4 copper layers, 90 x 90 mm, 95 parts, among them J1 JST-PH, J10 USB_C_USB2.0_16P, J11 Micro_SD_Card, J12 duPont, J2 JST-PH, J3 JST-PH, J4 duPont, J5 duPont, J6 duPont, J8 USB_C_USB2.0_16P, Q1 Si2301CDS, Q2 Si2301CDS, SW11 SW_QSPI, SW12 SW_RUN, SW3 SW_GNSS, U11 W25Q128JVS, U12 RP2350_60QFN, U3 TPS63001DRCR, U4 BH-18650-A6AJ012, U5 E32-400M30S, U6 NEO-M9N, Y11 ABM8_262_T3

Commit message: v1.0.1 - RF Fix
Routing:
- added copper zone on In1.Cu, net +1V1
Changed lines of the file:
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@@
 	)
 	(via
-		(at 158.75 69.65)
+		(at 158.6 69.8)
 		(size 0.6)
 		(drill 0.3)
@@
 	)
 	(via
-		(at 156 71)
+		(at 156.2 71)
 		(size 0.6)
 		(drill 0.3)
@@
 	)
 	(via
-		(at 156 72.35)
+		(at 156.2 72.2)
 		(size 0.6)
 		(drill 0.3)
@@
 	)
 	(via
-		(at 158.75 72.35)
+		(at 158.6 72.2)
 		(size 0.6)
 		(drill 0.3)
@@
 	)
 	(via
-		(at 156 69.65)
+		(at 156.2 69.8)
 		(size 0.6)
 		(drill 0.3)
@@
 	)
 	(via
-		(at 157.375 69.65)
+		(at 157.375 69.8)
 		(size 0.6)
 		(drill 0.3)
@@
 	)
 	(via
-		(at 158.75 71)
+		(at 158.6 71)
 		(size 0.6)
 		(drill 0.3)
@@
 	)
 	(via
-		(at 157.375 72.35)
+		(at 157.375 72.2)
 		(size 0.6)
 		(drill 0.3)
@@
 		(start 139.23 84)
 		(end 140.35 85.12)
-		(width 0.2)
+		(width 0.15)
 		(layer "F.Cu")
 		(net 32)
@@
 		(start 136.5 84)
 		(end 139.23 84)
-		(width 0.2)
+		(width 0.15)
 		(layer "F.Cu")
 		(net 32)
 	)
 	(segment
-		(start 140.3 82.53)
-		(end 140.35 82.58)
+		(start 136.5 82)
+		(end 139.77 82)
 		(width 0.15)
 		(layer "F.Cu")
@@
 	)
 	(segment
-		(start 139.77 82)
-		(end 140.35 82.58)
-		(width 0.2)
-		(layer "F.Cu")
-		(net 33)
-	)
-	(segment
-		(start 136.5 82)
+		(start 140.35 82.58)
 		(end 139.77 82)
-		(width 0.2)
+		(width 0.15)
 		(layer "F.Cu")
 		(net 33)
@@
 	)
 	(zone
-		(net 3)
-		(net_name "+1V1")
+		(net 25)
+		(net_name "GND")
 		(layer "B.Cu")
+		(name "GND")
 		(hatch edge 0.5)
-		(priority 12)
-		(connect_pads
+		(connect_pads yes
 			(clearance 0.3)
 		)
@@
 			(thermal_gap 0.5)
 			(thermal_bridge_width 0.5)
+			(smoothing fillet)
+			(radius 0.1)
 		)
 		(polygon
 			(pts
-				(xy 156.975 63.1) (xy 156.975 64.994872) (xy 153.175 68.6) (xy 152.175 69.6) (xy 152.175 70.5) (xy 155.375 70.5)
-				(xy 155.375 69) (xy 159.375 69) (xy 159.375 73) (xy 157.275 73) (xy 157.275 76.7) (xy 158.275 76.7)
-				(xy 162.675 72.3) (xy 162.675 70.3) (xy 157.975 65.6) (xy 157.975 63.1)
+				(xy 130 40) (xy 220 40) (xy 220 130) (xy 130 130)
 			)
 		)
 	)
 	(zone
-		(net 25)
-		(net_name "GND")
-		(layer "B.Cu")
-		(name "GND")
+		(net 3)
+		(net_name "+1V1")
+		(layers "B.Cu" "In1.Cu")
 		(hatch edge 0.5)
-		(connect_pads yes
+		(priority 12)
+		(connect_pads
 			(clearance 0.3)
 		)
@@
 			(thermal_gap 0.5)
 			(thermal_bridge_width 0.5)
-			(smoothing fillet)
-			(radius 0.1)
 		)
 		(polygon
 			(pts
-				(xy 130 40) (xy 220 40) (xy 220 130) (xy 130 130)
+				(xy 156.975 63.1) (xy 156.975 64.994872) (xy 153.175 68.6) (xy 152.175 69.6) (xy 152.175 70.5) (xy 155.375 70.5)
+				(xy 155.375 69) (xy 159.375 69) (xy 159.375 73) (xy 157.275 73) (xy 157.275 76.7) (xy 158.275 76.7)
+				(xy 162.675 72.3) (xy 162.675 70.3) (xy 157.975 65.6) (xy 157.975 63.1)
 			)
 		)

Commit message: v1.0.1
Parts:
- moved C19 0.40 mm to (163.5, 70.0)
- moved C24 0.40 mm to (163.5, 71.0)
Connections:
- U12 pad 34: /MCU/RF_RXEN -> /MCU/RF_IRQ
- U12 pad 35: /MCU/RF_TXEN -> /MCU/RF_RXEN
- U12 pad 36: unconnected-(U12-GPIO24-Pad36) -> /MCU/RF_TXEN
- U5 pad 20: unconnected-(U5-DIO0-Pad20) -> /MCU/RF_IRQ
Routing:
- net /MCU/RF_IRQ: track 0.00 -> 7.76 mm
- net /MCU/RF_RXEN: track 34.7 -> 34.9 mm, vias 0 -> 2

Commit message: init v1.0.2
Connections:
- J11 pad 2: /GNSS & MicroSD/SPI_CS1 -> /GNSS & MicroSD/SPI_CS0
- SW12 pad 2: +3V3 -> Net-(U12-RUN)
- U12 pad 15: /GNSS & MicroSD/SPI_CS1 -> /GNSS & MicroSD/SPI_CS0
- U12 pad 17: /GNSS & MicroSD/SPI_CS0 -> /GNSS & MicroSD/SPI_CS1
- U12 pad 26: +3V3 -> Net-(U12-RUN)
- U5 pad 19: unconnected-(U5-DIO1-Pad19) -> /RF/DIO1
- U5 pad 8: unconnected-(U5-DI02-Pad8) -> /RF/DI02
- U6 pad 1: Net-(U6-~{SAFEBOOT}) -> unconnected-(U6-~{SAFEBOOT}-Pad1)
- U6 pad 14: unconnected-(U6-LNA_EN-Pad14) -> /GNSS & MicroSD/LNA_EN
- U6 pad 18: /GNSS & MicroSD/SPI_CS0 -> /GNSS & MicroSD/SPI_CS1
- U6 pad 3: unconnected-(U6-TIMEPULSE-Pad3) -> /GNSS & MicroSD/TIMEPULSE
- U6 pad 4: unconnected-(U6-EXTINT-Pad4) -> /GNSS & MicroSD/EXTINT
Routing:
- net +3V3: track 59.5 -> 34.8 mm
- net Net-(U12-RUN): track 0.00 -> 24.7 mm
- net /GNSS & MicroSD/SPI_CS1: track 37.5 -> 46.2 mm, vias 0 -> 2
- net /GNSS & MicroSD/SPI_CS0: track 46.2 -> 37.5 mm, vias 2 -> 0
- net /MCU/QSPI_SD0: track 7.83 -> 8.91 mm
- net /MCU/RF_TXEN: track 34.0 -> 34.5 mm, vias 0 -> 2
- net GND: vias 333 -> 332

Commit message: v1.0.2 changelog
Parts:
- removed TP1: nSAFEBOOT, TestPoint:TestPoint_Pad_D1.0mm
- removed TP3: +3V3, TestPoint:TestPoint_Pad_D1.0mm
- removed TP4: GND, TestPoint:TestPoint_Pad_D1.0mm
- added D1: SMF3.3CA, Diode_SMD:D_SOD-123FL, F.Cu at (139.0, 85.6)
- added D2: SMF3.3CA, Diode_SMD:D_SOD-123FL, F.Cu at (139.0, 80.5)
- added D31: KT-0805W, LED_SMD:LED_0805_2012Metric, F.Cu at (169.0, 43.0)
- added D32: KT-0805W, LED_SMD:LED_0805_2012Metric, F.Cu at (193.3, 43.1)
- added G***: LOGO, silkscreens:BLV_v1_QR, F.Cu at (164.5, 54.5)
- added J31: PinHeader_01x02_Pin, Connector_PinHeader_2.54mm:PinHeader_1x02_P2.54mm_Vertical, F.Cu at (144.8, 125.0)
- added R1: 10k, Resistor_SMD:R_0402_1005Metric, F.Cu at (154.0, 97.6)
- added R2: 10k, Resistor_SMD:R_0402_1005Metric, F.Cu at (150.3, 75.0)
- added R36: 2k, Resistor_SMD:R_0603_1608Metric, F.Cu at (166.5, 44.4)
- added R37: 2k, Resistor_SMD:R_0603_1608Metric, F.Cu at (192.3, 45.8)
- added TP61: TestPoint, TestPoint:TestPoint_THTPad_D1.5mm_Drill0.7mm, F.Cu at (170.0, 125.0)
- added TP62: TestPoint, TestPoint:TestPoint_THTPad_D1.5mm_Drill0.7mm, F.Cu at (170.0, 122.0)
- added TP63: TestPoint, TestPoint:TestPoint_THTPad_D1.5mm_Drill0.7mm, F.Cu at (170.0, 128.0)
- added TP64: TestPoint, TestPoint:TestPoint_THTPad_D1.5mm_Drill0.7mm, F.Cu at (155.2, 107.2)
- added TP65: TestPoint, TestPoint:TestPoint_THTPad_D1.5mm_Drill0.7mm, F.Cu at (143.0, 93.0)
- added TP66: TestPoint, TestPoint:TestPoint_THTPad_D1.5mm_Drill0.7mm, F.Cu at (137.0, 113.0)
- D11, D12, D13: value GREEN -> KT-0805G
- D4: value GREEN -> KT0805Y
- R26, R27, R28: value 470 -> 1k
- R35: value 1k -> 2k
- SW11: value SW_QSPI -> SW_Push; footprint Button_Switch_SMD:SW_SPST_B3U-1000P -> Button_Switch_SMD:SW_Push_1P1T_NO_CK_KMR2
- SW12: value SW_RUN -> SW_Push; footprint Button_Switch_SMD:SW_SPST_B3U-1000P -> Button_Switch_SMD:SW_Push_1P1T_NO_CK_KMR2
- SW61: renamed from SW3; footprint Button_Switch_SMD:SW_SPST_B3U-1000P -> Button_Switch_SMD:SW_Push_1P1T_NO_CK_KMR2
- moved R66 3.91 mm to (186.0, 112.5), turned to 90 degrees
- moved C65 2.54 mm to (134.9, 94.4)
- moved C66 2.54 mm to (137.7, 94.9)
- moved R15 2.29 mm to (155.6, 93.5), turned to 0 degrees
- moved R20 1.84 mm to (142.0, 79.0)
- moved R24 1.75 mm to (143.5, 79.0)
- moved J6 1.31 mm to (141.5, 87.0)
- moved SW11 1.00 mm to (146.0, 48.3)
- moved SW61 0.71 mm to (182.5, 112.5), turned to 0 degrees
- moved SW12 0.30 mm to (158.5, 95.5), turned to 90 degrees
- moved R17 0.15 mm to (144.9, 54.5)
- turned J62 to 90 degrees
- renumbered C60 to C61, C61 to C62, C62 to C63, C67 to C64, J10 to J61, J11 to J62, JP1 to JP61, L67 to L61, R62 to R61, R63 to R62, R67 to R63, R60 to R64, R61 to R65, R64 to R66, U5 to U51, U6 to U61
Connections:
- net Net-(U12-RUN) renamed /MCU/RUN
- J62 pad 1: unconnected-(J11-DAT2-Pad1) -> /GNSS & MicroSD/DAT2
- J62 pad 8: unconnected-(J11-DAT1-Pad8) -> /GNSS & MicroSD/DAT1
- U51 pad 19: /RF/DIO1 -> unconnected-(U51-DIO1-Pad19)
- U51 pad 8: /RF/DI02 -> unconnected-(U51-DI02-Pad8)
- U61 pad 1: unconnected-(U6-~{SAFEBOOT}-Pad1) -> /GNSS & MicroSD/~{SAFEBOOT}
Routing:
- net /GNSS & MicroSD/DAT1: track 0.00 -> 8.64 mm
- net /GNSS & MicroSD/~{SAFEBOOT}: track 0.00 -> 6.66 mm
- net /GNSS & MicroSD/DAT2: track 0.00 -> 6.50 mm
- net /GNSS & MicroSD/LNA_EN: track 0.00 -> 6.45 mm, vias 0 -> 1
- net /GNSS & MicroSD/TIMEPULSE: track 0.00 -> 6.26 mm
- net /GNSS & MicroSD/EXTINT: track 0.00 -> 5.47 mm
- net /GNSS & MicroSD/SPI_CS0: track 37.5 -> 42.9 mm, vias 0 -> 2
- net /GNSS & MicroSD/SPI_MOSI: track 63.2 -> 68.1 mm
- net /GNSS & MicroSD/SPI_MISO: track 58.8 -> 63.3 mm
- net /GNSS & MicroSD/SPI_SCK: track 68.7 -> 73.1 mm
- net /MCU/SW_RUN_R: track 1.52 -> 5.71 mm
- net /GNSS & MicroSD/GNSS_RST_R: track 1.50 -> 5.67 mm
- net /MCU/~{USB_BOOT}: track 5.00 -> 8.35 mm
- net /GNSS & MicroSD/GNSS_RST: track 18.2 -> 21.3 mm
- net Net-(U6-~{SAFEBOOT}): track 2.32 -> 0.00 mm
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Other:
- board text added: "3V3"
- board text added: "BLV Data, Telemetry, and LoRaLink Board V1.0 by Tri Do"
- board text added: "BLVLink v1.0"
- board text removed: "BLV PCB v0.1"
- board text removed: "Designed by Tri Do"

Commit message: safepoint
Parts:
- D4: value KT0805Y -> KT-0805Y
- J12, J4, J5, J6: value duPont -> PinHeader_01x03_Pin
- L61: footprint Inductor_SMD:L_0201_0603Metric -> Inductor_SMD:L_0402_1005Metric
- SW11, SW12: value SW_Push -> KMR2
- SW61: value SW_GNSS -> KMR2
- moved J6 0.50 mm to (142.0, 87.0)
- moved R63 0.42 mm to (168.0, 115.2)
- moved D1 0.30 mm to (139.3, 85.6)
- moved D2 0.30 mm to (139.3, 80.5)
- moved C64 0.30 mm to (168.1, 113.7)
- moved L61 0.10 mm to (168.6, 112.2)
Routing:
- net /GNSS & MicroSD/SPI_SCK: track 73.1 -> 70.2 mm
- net /GNSS & MicroSD/GNSS_RST: track 21.3 -> 22.1 mm
- net /MCU/RUN: track 26.9 -> 26.1 mm
- net /GNSS & MicroSD/RF_BIAS_T: track 2.49 -> 3.10 mm
- net GND: vias 327 -> 325
- net +3V3: vias 44 -> 42

Commit message: v1.0.2 Fab
Routing:
- net GND: vias 325 -> 331

Commit message: Post-manufacturing v1 check.
Parts:
- removed G***: LOGO, silkscreens:BLV_v1_QR
- C61: value 10uF -> 10u
- C62: value 1uF -> 1u
- moved R30 0.30 mm to (155.0, 50.2)
- moved R31 0.30 mm to (158.0, 50.2)
Routing:
- net GND: track 17.0 -> 18.7 mm, vias 331 -> 333
Other:
- board text added: "BLVLink v2.0"
- board text removed: "BLVLink v1.0"

Commit message: 3/18 nightly build
Parts:
- removed D31, D32: KT-0805W, LED_SMD:LED_0805_2012Metric
- removed R36, R37: 2k, Resistor_SMD:R_0603_1608Metric
Routing:
- net /Power/BATT_LED: track 1.90 -> 0.00 mm
- net /Power/VUSB_LED: track 1.80 -> 0.00 mm
- net GND: track 18.7 -> 17.3 mm
Other:
- board text added: "+"
- board text added: "-"
- board text added: "BLV Data, Telemetry, and LoRaLink Board by Tri Do"
- board text added: "Funded with hopes and dreams"
- board text removed: "BLV Data, Telemetry, and LoRaLink Board V1.0 by Tri Do"
- board text removed: "Funded with hope and dreams"
