File: Power.kicad_sch (KiCad schematic)
At the start: 21 parts, among them J8 USB_C_USB2.0_16P, Q1 Si2301CDS, Q2 Si2301CDS, U3 TPS63001DRCR, U4 BH-18650-A6AJ012

Commit message: init v1.0.2
Parts:
- R35: value 1k -> 2k
Other:
- title: +5V, +3V3, LiPo Battery, Charger -> +3V3, LiPo Battery
Changed lines of the file:
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@@
 	(paper "USLedger")
 	(title_block
-		(title "+5V, +3V3, LiPo Battery, Charger")
-		(date "2025-11-11")
-		(rev "C")
+		(title "+3V3, LiPo Battery")
+		(date "2026-03-05")
+		(rev "v1.0.2")
 		(company "Bronco STAR - BLV")
-		(comment 1 "Rev B - Add TP4056 Charger, Line Switcher, +5V SMPS")
-		(comment 2 "Rev C - Remove LiPo Charger due to not recommended IC. Implement PMOS Ideal Diode.")
+		(comment 1 "PMOS Ideal Diode Source Switching")
 	)
 	(rectangle
@@
 			)
 		)
-		(property "Value" "1k"
+		(property "Value" "2k"
 			(at 293.37 99.06 90)
 			(effects

Commit message: v1.0.2 changelog
Parts:
- removed TP3: +3V3, TestPoint:TestPoint_Pad_D1.0mm, symbol Connector:TestPoint
- removed TP4: GND, TestPoint:TestPoint_Pad_D1.0mm, symbol Connector:TestPoint
- added D31, D32: KT-0805W, LED_SMD:LED_0805_2012Metric, symbol Device:LED
- added J31: PinHeader_01x02_Pin, Connector_PinHeader_2.54mm:PinHeader_1x02_P2.54mm_Vertical, symbol Connector:Conn_01x02_Pin
- added R36, R37: 2k, Resistor_SMD:R_0603_1608Metric, symbol Device:R
- D4: value GREEN -> KT-0805Y
Connections:
- net +3V3: now also J31.1 (Pin_1)
- net +BATT: now also R37.1
- net GND: now also D31.1 (K), D32.1 (K), J31.2 (Pin_2)
- net VBUS: now also R36.1
- new net BATT_LED: D32.2 (A), R37.2
- new net VUSB_LED: D31.2 (A), R36.2
Other:
- moved on the sheet: U4

Commit message: Post-manufacturing v1 check.
Parts:
- C30, C31, C33: LCSC Part C1525 -> (none)
Changed lines of the file:
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@@
 			)
 		)
-		(property "LCSC Part" "C1525"
+		(property "LCSC Part" ""
 			(at 214.63 111.76 0)
 			(effects
@@
 			)
 		)
-		(property "LCSC Part" "C1525"
+		(property "LCSC Part" ""
 			(at 132.08 68.58 0)
 			(effects
@@
 			)
 		)
-		(property "LCSC Part" "C1525"
+		(property "LCSC Part" ""
 			(at 132.08 132.08 0)
 			(effects

Commit message: 3/18 nightly build
Parts:
- removed D31, D32: KT-0805W, LED_SMD:LED_0805_2012Metric, symbol Device:LED
- removed R36, R37: 2k, Resistor_SMD:R_0603_1608Metric, symbol Device:R

Commit message: discrete protection, charger, ideal diodes, and 5v smps
Parts:
- removed Q1, Q2: Si2301CDS, Package_TO_SOT_SMD:SOT-23, symbol Transistor_FET:DMG2301L
- added C? (x2): 1u, symbol Device:C
- added C?: 0.1u, symbol Device:C
- added D? (x3): LED, symbol Device:LED
- added Q? (x2): CSD16406Q3, Package_TO_SOT_SMD:TDSON-8-1, symbol Transistor_FET:CSD16404Q5A
- added Q? (x2): AO3401A, Package_TO_SOT_SMD:SOT-23, symbol Transistor_FET:AO3401A
- added R?: 10k, symbol Device:R
- added R?: 330, symbol Device:R
- added R? (x3): 1.5k, symbol Device:R
- added R?: 2.2k, symbol Device:R
- added R?: 2k, symbol Device:R
- added SW?: SW_SPDT, symbol Switch:SW_SPDT
- added U?: BQ29707, Package_SON:WSON-6_1.5x1.5mm_P0.5mm, symbol Battery_Management:BQ297xy
- added U?: INA260, Package_SO:TSSOP-16_4.4x5mm_P0.65mm, symbol Sensor:INA260
- added U?: MCP73833-xxx-MF, Package_DFN_QFN:DFN-10-1EP_3x3mm_P0.5mm_EP1.58x2.35mm, symbol Battery_Management:MCP73833-xxx-MF
- L2: value 2u2 -> VLS4012ET-2R2M
Connections:
- net +3V3: now also U?.10 (VS)
- net GND: now also C?.2, C?.2, Q?.1 (S), Q?.2 (S), Q?.3 (S), R?.2, R?.2, R?.2, U?.11 (EP), U?.11 (GND), U?.4 (A1), U?.5 (A0), U?.5 (V_{SS}), U?.6 (GND); no longer U4.1
- net VBUS: now also C?.1, D?.2 (A), D?.2 (A), D?.2 (A), Q?.2 (S), U?.1 (V_{DD}), U?.2 (V_{DD})
- net +BATT renamed CELL+
- net CELL+: now also C?.1, Q?.2 (S), R?.1, U?.10 (V_{BAT}), U?.9 (V_{BAT})
- net Vin: no longer names the net of C30.2, C31.2, R32.1, R33.1
- net Vin: now also Q?.1 (G), Q?.1 (G), Q?.3 (D), Q?.3 (D), SW?.2 (B); no longer C32.1, R34.1, U3.5 (VIN)
- new net: Q?.5 (D), Q?.5 (D)
- new net: C32.1, R34.1, U3.5 (VIN), U?.14 (IN-), U?.15 (IN-), U?.16 (IN-)
- new net: SW?.3 (C), U?.1 (IN+), U?.12 (VBUS), U?.2 (IN+), U?.3 (IN+)
- new net BAT: C?.1, R?.2, U?.5 (BAT)
- new net CELL-: C?.2, Q?.1 (S), Q?.2 (S), Q?.3 (S), U4.1, U?.4 (VSS)
- new net Cout: Q?.4 (G), U?.2 (Cout)
- new net Dout: Q?.4 (G), U?.3 (Dout)
- new net I2C0_SCL: U?.9 (SCL)
- new net I2C0_SDA: U?.8 (SDA)
- new net PROG: R?.1, U?.6 (PROG)
- new net R_PG: D?.1 (K), R?.1
- new net R_STAT1: D?.1 (K), R?.1
- new net R_STAT2: D?.1 (K), R?.1
- new net STAT1: R?.2, U?.3 (STAT1)
- new net STAT2: R?.2, U?.4 (STAT2)
- new net THERM: R?.1, U?.8 (THERM)
- new net V-: R?.1, U?.6 (V-)
- new net ~{PG}: R?.2, U?.7 (~{PG})
- no-connect marks 3 -> 4
Other:
- note added: "Battery Charger"
- note added: "Battery Protection"
- note added: "I2C address = 0x40"
- note added: "Power Monitor I/V/P"
- note added: "Rprog = 1000V / Ireg"
- note added: "SMPS +5V @ ?A Boost"
- note added: "STAT1 = CHARGE IN PROGRESS STAT2 = CHARGE COMPLETE PG = POWER TO CHARGER"
- note added: "System ON/OFF SW"
- note added: "USB-C (RP2350)"
- note added: "overcharge, overdischarge, overcurrent, short-circuit protection"
- note removed: "No on-board charging. Use external charger"
- note removed: "USB-C"
- moved on the sheet: C30, C31, C32, C33, C34, C35, D4, J31, J8, L2, R30, R31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

Commit message: rough power layout
Parts:
- removed Q? (x2): AO3401A, Package_TO_SOT_SMD:SOT-23, symbol Transistor_FET:AO3401A
- added Q3, Q4: CSD25402Q3A, Package_SON:VSON-8_3.3x3.3mm_P0.65mm_NexFET, symbol Transistor_FET:CSD25402Q3A
- gave numbers to parts that had none: 19
Connections:
- net CELL+: now also Q4.5 (S)
- net VBUS: now also Q3.5 (S)
- net Monitor_out: now reaches C32.1, R34.1, U3.5 (VIN), U6.14 (IN-), U6.15 (IN-), U6.16 (IN-)
- net Monitor_in: now reaches SW1.3 (C), U6.1 (IN+), U6.12 (VBUS), U6.2 (IN+), U6.3 (IN+)
- net V_SWITCH: now reaches C30.2, C31.2, R32.1, R33.1, SW1.2 (B)
- net V_SWITCH: now also Q3.1 (D), Q3.2 (D), Q3.3 (D), Q3.4 (G), Q4.1 (D), Q4.2 (D), Q4.3 (D), Q4.4 (G)
Other:
- moved on the sheet: Q2

Commit message: 050326 layouts
Parts:
- removed SW1: SW_SPDT, symbol Switch:SW_SPDT
- added C36: 10u, Capacitor_SMD:C_0603_1608Metric, symbol Device:C
- added C38: 1u, Capacitor_SMD:C_0402_1005Metric, symbol Device:C
- added C40: 10p, Capacitor_SMD:C_0402_1005Metric, symbol Device:C
- added C41, C43, C45: 22u, Capacitor_SMD:C_0805_2012Metric, symbol Device:C
- added D34: KT-0805G, LED_SMD:LED_0805_2012Metric, symbol Device:LED
- added L31: XAL7030-102ME, Inductor_SMD:L_Coilcraft_XAL7030-102, symbol Device:L
- added R43: 1M, Resistor_SMD:R_0402_1005Metric, symbol Device:R
- added R44: 330k, Resistor_SMD:R_0402_1005Metric, symbol Device:R
- added R45: 2k, Resistor_SMD:R_0603_1608Metric, symbol Device:R
- added SW31: K3-1391B-51, Slide_Switch:SW-TH_K3-1391B-51, symbol Slide_Switch:K3-1391B-51
- added U35: TPS61236PRWLR, TPS61236:VQFN-9_L2.5-W2.5-P0.50-TL, symbol TPS61236:TPS61236PRWLR
- C31: renamed from C1; footprint (none) -> Capacitor_SMD:C_0402_1005Metric
- C32: renamed from C2; footprint (none) -> Capacitor_SMD:C_0603_1608Metric
- C33: renamed from C3; footprint (none) -> Capacitor_SMD:C_0603_1608Metric
- D31: renamed from D3; footprint (none) -> LED_SMD:LED_0805_2012Metric
- D32: renamed from D5; footprint (none) -> LED_SMD:LED_0805_2012Metric
- D33: renamed from D6; footprint (none) -> LED_SMD:LED_0805_2012Metric
- R31: renamed from R3; footprint (none) -> Resistor_SMD:R_0603_1608Metric
- R34: renamed from R4; footprint (none) -> Resistor_SMD:R_0402_1005Metric
- R35: renamed from R5; value 1.5k -> 2k; footprint (none) -> Resistor_SMD:R_0402_1005Metric
- R36: renamed from R6; value 1.5k -> 2k; footprint (none) -> Resistor_SMD:R_0402_1005Metric
- R37: renamed from R7; value 1.5k -> 2k; footprint (none) -> Resistor_SMD:R_0402_1005Metric
- R38: renamed from R8; footprint (none) -> Resistor_SMD:R_0402_1005Metric
- R39: renamed from R9; footprint (none) -> Resistor_SMD:R_0402_1005Metric
- U33: renamed from U2; value MCP73833-xxx-MF -> MCP73833-FCI-MF
- renumbered C30 to C34, C31 to C35, C32 to C37, C33 to C39, C34 to C42, C35 to C44, D4 to D35, J8 to J31, J31 to J32, L2 to L32, Q1 to Q31, Q2 to Q32, Q3 to Q33, Q4 to Q34, R30 to R32, R31 to R33, R32 to R40, R33 to R41, R34 to R42, R35 to R46, U4 to U31, U1 to U32, U6 to U34, U3 to U36
Connections:
- net GND: now also C36.2, C38.2, C41.2, C43.2, C45.2, D34.1 (K), R44.2, U35.1 (PGND), U35.4 (CC), U35.5 (AGND), U35.8 (INACT)
- net Monitor_in: now also SW31.3
- net Monitor_out: now also C36.1, C38.1, L31.1, U35.3 (VIN), U35.7 (EN)
- net V_SWITCH: now also SW31.2
- new net +5V: C40.1, C41.1, C43.1, C45.1, R43.1, R45.1, U35.9 (VOUT)
- new net 5V_LED: D34.2 (A), R45.2
- new net FB: C40.2, R43.2, R44.1, U35.6 (FB)
- new net SW: L31.2, U35.2 (SW)
- no-connect marks 4 -> 5
Other:
- note added: "FB Network: 1.244 * (1 + 1M / 330k) = 5.014 V"
- note added: "SMPS +5V @ 5A Boost"
- note removed: "SMPS +5V @ ?A Boost"
- moved on the sheet: C32, C33, D35, R46, U34
