File: Sensors.kicad_sch (KiCad schematic)
At the start: 0 parts

Commit message: v2 layouts done
Parts:
- added C71: 100n, Capacitor_SMD:C_0402_1005Metric, symbol Device:C
- added U71: MCP9808_DFN, Package_DFN_QFN:DFN-8-1EP_3x2mm_P0.5mm_EP1.7x1.4mm, symbol Sensor_Temperature:MCP9808_DFN
Connections:
- new net +3V3: C71.1, U71.8 (V_{DD})
- new net GND: C71.2, U71.4 (GND), U71.5 (A2), U71.6 (A1), U71.7 (A0), U71.9 (EP/GND)
- new net I2C0_SCL: U71.2 (SCL)
- new net I2C0_SDA: U71.1 (SDA)
- no-connect marks 0 -> 1
Other:
- note added: "I2C address = 0x18"
- note added: "Temp Sensor"
- note removed: "Temp Sensor?"
